File: Rpi5/PCB/SensorBoxPython.kicad_pcb (KiCad board)
At the start: 2 copper layers, 65 x 56 mm, 9 parts, among them J1 GPIO

Commit message: PCB Files
Parts:
- moved C2 19.1 mm to (117.5, 92.0)
Connections:
- AHT20+BMP280 pad 2: Net-(AHT20+BMP280-SDA) -> /ID_SDA
- AHT20+BMP280 pad 4: Net-(AHT20+BMP280-SCL) -> /ID_SCL
- PMS5003 pad 3: unconnected-(PMS5003-SET-Pad3) -> /GPIO3/SCL1
- PMS5003 pad 4: unconnected-(PMS5003-RXD-Pad4) -> /GPIO14/TXD0
- PMS5003 pad 5: unconnected-(PMS5003-TXD-Pad5) -> /GPIO15/RXD0
- PMS5003 pad 6: unconnected-(PMS5003-RST-Pad6) -> /GPIO2/SDA1
- SGP30 pad 3: Net-(AHT20+BMP280-SDA) -> /ID_SDA
- SGP30 pad 4: Net-(AHT20+BMP280-SCL) -> /ID_SCL
Routing:
- net /ID_SCL: track 0.00 -> 44.8 mm
- net Net-(AHT20+BMP280-SCL): track 34.6 -> 0.00 mm
- net /GPIO3/SCL1: track 0.00 -> 31.1 mm
- net /ID_SDA: track 0.00 -> 27.5 mm
- net /GPIO14/TXD0: track 0.00 -> 23.7 mm
- net GND: track 109.6 -> 133.3 mm
- net Net-(AHT20+BMP280-SDA): track 21.1 -> 0.00 mm
- net /GPIO15/RXD0: track 0.00 -> 17.6 mm
- net /GPIO2/SDA1: track 0.00 -> 16.5 mm
- net +5V: track 106.6 -> 118.9 mm
- net unconnected-(PMS5003-RST-Pad6): track 8.29 -> 0.00 mm
- net unconnected-(PMS5003-RXD-Pad4): track 8.26 -> 0.00 mm
- net unconnected-(PMS5003-TXD-Pad5): track 8.07 -> 0.00 mm
- net unconnected-(PMS5003-SET-Pad3): track 8.03 -> 0.00 mm
Other:
- board text added: "AHT20+BMP280"
- board text added: "SensorBox V1.0 Jonas Bouchard"
