File: Rpi5/PCB/SensorBoxPython.kicad_sch (KiCad schematic)
At the start: 10 parts, among them J1 GPIO, U1 CAT24C256

Commit message: PCB Files
Connections:
- net GPIO14/TXD0: now also PMS5003.4 (RXD)
- net GPIO15/RXD0: now also PMS5003.5 (TXD)
- net GPIO2/SDA1: now also PMS5003.6 (RST)
- net GPIO3/SCL1: now also PMS5003.3 (SET)
- net ID_SCL: now also AHT20+BMP280.4 (SCL), SGP30.4 (SCL)
- net ID_SDA: now also AHT20+BMP280.2 (SDA), SGP30.3 (SDA)
Changed lines of the file:
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@@
+	)
+	(junction
+		(at 146.05 41.91)
+		(diameter 0)
+		(color 0 0 0 0)
 	)
 	(junction
@@
 	)
 	(junction
+		(at 142.24 80.01)
+		(diameter 0)
+		(color 0 0 0 0)
+	)
+	(junction
 		(at 205.74 99.06)
 		(diameter 1.016)
@@
 	(wire
 		(pts
+			(xy 233.68 116.84) (xy 233.68 73.66)
+		)
+		(stroke
+			(width 0)
+			(type default)
+		)
+	)
+	(wire
+		(pts
 			(xy 190.5 76.2) (xy 161.29 76.2)
 		)
@@
 	(wire
 		(pts
+			(xy 236.22 119.38) (xy 236.22 71.12)
+		)
+		(stroke
+			(width 0)
+			(type default)
+		)
+	)
+	(wire
+		(pts
 			(xy 205.74 68.58) (xy 205.74 78.74)
 		)
@@
 	(wire
 		(pts
+			(xy 125.73 116.84) (xy 233.68 116.84)
+		)
+		(stroke
+			(width 0)
+			(type default)
+		)
+	)
+	(wire
+		(pts
 			(xy 125.73 44.45) (xy 130.81 44.45)
 		)
@@
 	(wire
 		(pts
+			(xy 149.86 96.52) (xy 190.5 96.52)
+		)
+		(stroke
+			(width 0)
+			(type default)
+		)
+	)
+	(wire
+		(pts
 			(xy 205.74 86.36) (xy 205.74 99.06)
 		)
@@
 	(wire
 		(pts
-			(xy 203.2 71.12) (xy 229.87 71.12)
+			(xy 203.2 71.12) (xy 236.22 71.12)
 		)
 		(stroke
@@
 	(wire
 		(pts
-			(xy 190.5 96.52) (xy 161.29 96.52)
-		)
-		(stroke
-			(width 0)
-			(type solid)
-		)
-	)
-	(wire
-		(pts
 			(xy 130.81 44.45) (xy 130.81 27.94)
 		)
@@
 	(wire
 		(pts
-			(xy 161.29 68.58) (xy 190.5 68.58)
-		)
-		(stroke
-			(width 0)
-			(type solid)
-		)
-	)
-	(wire
-		(pts
 			(xy 161.29 91.44) (xy 190.5 91.44)
 		)
@@
 	(wire
 		(pts
+			(xy 157.48 68.58) (xy 190.5 68.58)
+		)
+		(stroke
+			(width 0)
+			(type default)
+		)
+	)
+	(wire
+		(pts
 			(xy 185.42 83.82) (xy 190.5 83.82)
 		)
@@
 	(wire
 		(pts
-			(xy 190.5 66.04) (xy 161.29 66.04)
-		)
-		(stroke
-			(width 0)
-			(type solid)
-		)
-	)
-	(wire
-		(pts
 			(xy 205.74 63.5) (xy 205.74 66.04)
 		)
@@
 	(wire
 		(pts
+			(xy 142.24 80.01) (xy 149.86 80.01)
+		)
+		(stroke
+			(width 0)
+			(type default)
+		)
+	)
+	(wire
+		(pts
+			(xy 149.86 80.01) (xy 149.86 96.52)
+		)
+		(stroke
+			(width 0)
+			(type default)
+		)
+	)
+	(wire
+		(pts
+			(xy 125.73 114.3) (xy 154.94 114.3)
+		)
+		(stroke
+			(width 0)
+			(type default)
+		)
+	)
+	(wire
+		(pts
 			(xy 125.73 127) (xy 133.35 127)
 		)
@@
 	(wire
 		(pts
+			(xy 243.84 41.91) (xy 243.84 96.52)
+		)
+		(stroke
+			(width 0)
+			(type default)
+		)
+	)
+	(wire
+		(pts
 			(xy 125.73 77.47) (xy 146.05 77.47)
 		)
@@
 	(wire
 		(pts
-			(xy 203.2 73.66) (xy 229.87 73.66)
+			(xy 203.2 73.66) (xy 233.68 73.66)
 		)
 		(stroke
@@
 	(wire
 		(pts
+			(xy 154.94 114.3) (xy 154.94 66.04)
+		)
+		(stroke
+			(width 0)
+			(type default)
+		)
+	)
+	(wire
+		(pts
+			(xy 146.05 41.91) (xy 243.84 41.91)
+		)
+		(stroke
+			(width 0)
+			(type default)
+		)
+	)
+	(wire
+		(pts
+			(xy 125.73 121.92) (xy 157.48 121.92)
+		)
+		(stroke
+			(width 0)
+			(type default)
+		)
+	)
+	(wire
+		(pts
 			(xy 161.29 81.28) (xy 190.5 81.28)
 		)
@@
 	(wire
 		(pts
+			(xy 125.73 119.38) (xy 236.22 119.38)
+		)
+		(stroke
+			(width 0)
+			(type default)
+		)
+	)
+	(wire
+		(pts
 			(xy 203.2 109.22) (xy 229.87 109.22)
 		)
@@
 	(wire
 		(pts
+			(xy 154.94 66.04) (xy 190.5 66.04)
+		)
+		(stroke
+			(width 0)
+			(type default)
+		)
+	)
+	(wire
+		(pts
 			(xy 125.73 82.55) (xy 130.81 82.55)
 		)
@@
 	(wire
 		(pts
+			(xy 157.48 121.92) (xy 157.48 68.58)
+		)
+		(stroke
+			(width 0)
+			(type default)
+		)
+	)
+	(wire
+		(pts
 			(xy 133.35 49.53) (xy 205.74 49.53)
 		)
@@
 	(wire
 		(pts
-			(xy 203.2 96.52) (xy 229.87 96.52)
-		)
-		(stroke
+			(xy 203.2 96.52) (xy 243.84 96.52)
+		)
+		(stroke
